File: Malfunctionboard UMCU.kicad_pcb (KiCad board)
At the start: 2 copper layers, 0 parts

Commit message: Changed: design to accomodate quad comparator package. Added: all labels for the connectors
Parts:
- added C101: 10n, Capacitor_SMD:C_0805_2012Metric, F.Cu at (338.3, 43.4)
- added C102: 10n, Capacitor_SMD:C_0805_2012Metric, F.Cu at (342.7, 43.4)
- added C103: 10n, Capacitor_SMD:C_0805_2012Metric, F.Cu at (330.1, 51.0)
- added C104: 10n, Capacitor_SMD:C_0805_2012Metric, F.Cu at (347.6, 34.6)
- added C105: 10n, Capacitor_SMD:C_0805_2012Metric, F.Cu at (316.8, 51.0)
- added C106: 10n, Capacitor_SMD:C_0805_2012Metric, F.Cu at (342.8, 36.2)
- added C107: 10n, Capacitor_SMD:C_0805_2012Metric, F.Cu at (333.9, 45.0)
- added C108: 10n, Capacitor_SMD:C_0805_2012Metric, F.Cu at (343.2, 33.3)
- added C109: 10n, Capacitor_SMD:C_0805_2012Metric, F.Cu at (352.0, 31.7)
- added C110: 10n, Capacitor_SMD:C_0805_2012Metric, F.Cu at (347.2, 37.6)
- added C111: 10n, Capacitor_SMD:C_0805_2012Metric, F.Cu at (333.9, 48.0)
- added C112: 10n, Capacitor_SMD:C_0805_2012Metric, F.Cu at (312.4, 51.0)
- added C113: 10n, Capacitor_SMD:C_0805_2012Metric, F.Cu at (347.6, 28.7)
- added C114: 10n, Capacitor_SMD:C_0805_2012Metric, F.Cu at (338.3, 40.5)
- added C115: 10n, Capacitor_SMD:C_0805_2012Metric, F.Cu at (325.7, 51.0)
- added C116: 10n, Capacitor_SMD:C_0805_2012Metric, F.Cu at (338.3, 46.4)
- added C117: 10n, Capacitor_SMD:C_0805_2012Metric, F.Cu at (347.6, 31.7)
- added C118: 10n, Capacitor_SMD:C_0805_2012Metric, F.Cu at (352.0, 28.7)
- added C119: 10n, Capacitor_SMD:C_0805_2012Metric, F.Cu at (342.7, 40.5)
- added C120: 10n, Capacitor_SMD:C_0805_2012Metric, F.Cu at (321.3, 51.0)
- added C201: 10n, Capacitor_SMD:C_0805_2012Metric, F.Cu at (359.1, 145.4)
- added C202: 10n, Capacitor_SMD:C_0805_2012Metric, F.Cu at (354.6, 148.9)
- added C203: 10n, Capacitor_SMD:C_0805_2012Metric, F.Cu at (359.1, 142.5)
- added C204: 10n, Capacitor_SMD:C_0805_2012Metric, F.Cu at (350.2, 147.4)
- added C205: 10n, Capacitor_SMD:C_0805_2012Metric, F.Cu at (345.8, 150.9)
- added C301: 10n, Capacitor_SMD:C_0805_2012Metric, F.Cu at (403.7, 64.2)
- added C302: 10n, Capacitor_SMD:C_0805_2012Metric, F.Cu at (408.1, 60.7)
- added C303: 10n, Capacitor_SMD:C_0805_2012Metric, F.Cu at (408.1, 66.6)
- added C304: 10n, Capacitor_SMD:C_0805_2012Metric, F.Cu at (417.0, 58.7)
- added C305: 10n, Capacitor_SMD:C_0805_2012Metric, F.Cu at (412.6, 65.1)
- added C401: 10n, Capacitor_SMD:C_0805_2012Metric, F.Cu at (374.9, 91.4)
- added C402: 10n, Capacitor_SMD:C_0805_2012Metric, F.Cu at (370.4, 95.9)
- added C403: 10n, Capacitor_SMD:C_0805_2012Metric, F.Cu at (374.9, 94.4)
- added C404: 10n, Capacitor_SMD:C_0805_2012Metric, F.Cu at (370.5, 90.0)
- added C405: 10n, Capacitor_SMD:C_0805_2012Metric, F.Cu at (374.9, 88.5)
- added C501: 10n, Capacitor_SMD:C_0805_2012Metric, F.Cu at (428.9, 39.2)
- added C502: 10n, Capacitor_SMD:C_0805_2012Metric, F.Cu at (424.5, 39.7)
- added C503: 10n, Capacitor_SMD:C_0805_2012Metric, F.Cu at (420.1, 44.1)
- added C504: 10n, Capacitor_SMD:C_0805_2012Metric, F.Cu at (428.9, 36.2)
- added C505: 10n, Capacitor_SMD:C_0805_2012Metric, F.Cu at (424.5, 42.6)
- added C601: 10n, Capacitor_SMD:C_0805_2012Metric, F.Cu at (370.5, 70.4)
- added C602: 10n, Capacitor_SMD:C_0805_2012Metric, F.Cu at (366.0, 73.9)
- added C603: 10n, Capacitor_SMD:C_0805_2012Metric, F.Cu at (378.1, 62.5)
- added C604: 10n, Capacitor_SMD:C_0805_2012Metric, F.Cu at (366.0, 70.9)
- added C605: 10n, Capacitor_SMD:C_0805_2012Metric, F.Cu at (379.3, 68.4)
- added C701: 10n, Capacitor_SMD:C_0805_2012Metric, F.Cu at (337.2, 88.5)
- added C702: 10n, Capacitor_SMD:C_0805_2012Metric, F.Cu at (337.2, 91.4)
- added C703: 10n, Capacitor_SMD:C_0805_2012Metric, F.Cu at (332.7, 95.9)
- added C704: 10n, Capacitor_SMD:C_0805_2012Metric, F.Cu at (337.2, 94.4)
- added C705: 10n, Capacitor_SMD:C_0805_2012Metric, F.Cu at (341.6, 90.9)
- added C801: 10n, Capacitor_SMD:C_0805_2012Metric, F.Cu at (386.8, 36.7)
- added C802: 10n, Capacitor_SMD:C_0805_2012Metric, F.Cu at (382.4, 41.2)
- added C803: 10n, Capacitor_SMD:C_0805_2012Metric, F.Cu at (382.4, 44.1)
- added C804: 10n, Capacitor_SMD:C_0805_2012Metric, F.Cu at (391.2, 36.2)
- added C805: 10n, Capacitor_SMD:C_0805_2012Metric, F.Cu at (382.4, 38.2)
- added C901: 10n, Capacitor_SMD:C_0805_2012Metric, F.Cu at (341.6, 68.4)
- added C902: 10n, Capacitor_SMD:C_0805_2012Metric, F.Cu at (341.6, 65.5)
- added C903: 10n, Capacitor_SMD:C_0805_2012Metric, F.Cu at (337.2, 71.9)
- added C904: 10n, Capacitor_SMD:C_0805_2012Metric, F.Cu at (332.8, 67.5)
- added C905: 10n, Capacitor_SMD:C_0805_2012Metric, F.Cu at (328.3, 70.9)
- added D101: 15V, Diode_SMD:D_SOD-323, F.Cu at (351.5, 37.6)
- added D102: 15V, Diode_SMD:D_SOD-323, F.Cu at (342.6, 46.4)
- added D103: 5V, Diode_SMD:D_SOD-323, F.Cu at (338.8, 49.3)
- added D104: 12V, Diode_SMD:D_SOD-323, F.Cu at (347.1, 43.5)
- added D105: 5.4V, Diode_SMD:D_SOD-323, F.Cu at (351.5, 40.5)
- added D106: 5.4V, Diode_SMD:D_SOD-323, F.Cu at (343.1, 49.3)
- added D107: 15V, Diode_SMD:D_SOD-323, F.Cu at (351.3, 43.5)
- added D201: LED, LED_SMD:LED_0805_2012Metric, F.Cu at (353.5, 140.0)
- added D202: LED, LED_SMD:LED_0805_2012Metric, F.Cu at (345.8, 144.9)
- added D301: LED, LED_SMD:LED_0805_2012Metric, F.Cu at (411.4, 56.2)
- added D302: LED, LED_SMD:LED_0805_2012Metric, F.Cu at (403.7, 61.2)
- added D401: LED, LED_SMD:LED_0805_2012Metric, F.Cu at (373.7, 85.5)
- added D402: LED, LED_SMD:LED_0805_2012Metric, F.Cu at (366.1, 90.4)
- added D501: LED, LED_SMD:LED_0805_2012Metric, F.Cu at (415.7, 38.7)
- added D502: LED, LED_SMD:LED_0805_2012Metric, F.Cu at (423.4, 33.7)
- added D601: LED, LED_SMD:LED_0805_2012Metric, F.Cu at (373.7, 63.0)
- added D602: LED, LED_SMD:LED_0805_2012Metric, F.Cu at (366.1, 67.9)
- added D701: LED, LED_SMD:LED_0805_2012Metric, F.Cu at (328.4, 90.4)
- added D702: LED, LED_SMD:LED_0805_2012Metric, F.Cu at (336.0, 85.5)
- added D801: LED, LED_SMD:LED_0805_2012Metric, F.Cu at (385.7, 33.7)
- added D802: LED, LED_SMD:LED_0805_2012Metric, F.Cu at (378.0, 38.7)
- added D901: LED, LED_SMD:LED_0805_2012Metric, F.Cu at (328.4, 67.9)
- added D902: LED, LED_SMD:LED_0805_2012Metric, F.Cu at (336.0, 63.0)
- added J101: Conn_02x05_Odd_Even, Connector_IDC:IDC-Header_2x05_P2.54mm_Vertical, F.Cu at (314.4, 33.4)
- added J102: Conn_02x05_Odd_Even, Connector_IDC:IDC-Header_2x05_P2.54mm_Vertical, F.Cu at (325.2, 33.4)
- added J201: Conn_Coaxial, _Custom:Solder straight thin coax cable, F.Cu at (336.8, 142.2)
- added J202: Conn_Coaxial, _Custom:Solder straight thin coax cable, F.Cu at (330.7, 142.2)
- added J301: Conn_Coaxial, _Custom:Solder straight thin coax cable, F.Cu at (388.6, 58.5)
- added J302: Conn_Coaxial, _Custom:Solder straight thin coax cable, F.Cu at (394.7, 58.5)
- added J401: Conn_Coaxial, _Custom:Solder straight thin coax cable, F.Cu at (351.0, 87.8)
- added J402: Conn_Coaxial, _Custom:Solder straight thin coax cable, F.Cu at (357.0, 87.8)
- added J501: Conn_Coaxial, _Custom:Solder straight thin coax cable, F.Cu at (400.6, 36.0)
- added J502: Conn_Coaxial, _Custom:Solder straight thin coax cable, F.Cu at (406.7, 36.0)
- added J601: Conn_Coaxial, _Custom:Solder straight thin coax cable, F.Cu at (357.0, 65.3)
- added J602: Conn_Coaxial, _Custom:Solder straight thin coax cable, F.Cu at (351.0, 65.3)
- added J701: Conn_Coaxial, _Custom:Solder straight thin coax cable, F.Cu at (319.4, 87.8)
- added J702: Conn_Coaxial, _Custom:Solder straight thin coax cable, F.Cu at (313.3, 87.8)
- added J801: Conn_Coaxial, _Custom:Solder straight thin coax cable, F.Cu at (369.0, 36.0)
- added J802: Conn_Coaxial, _Custom:Solder straight thin coax cable, F.Cu at (362.9, 36.0)
- added J901: Conn_Coaxial, _Custom:Solder straight thin coax cable, F.Cu at (313.3, 65.3)
- added J902: Conn_Coaxial, _Custom:Solder straight thin coax cable, F.Cu at (319.4, 65.3)
- added JP101: Jumper, Connector_PinHeader_2.54mm:PinHeader_1x02_P2.54mm_Vertical, F.Cu at (334.0, 29.6)
- added JP102: Jumper, Connector_PinHeader_2.54mm:PinHeader_1x02_P2.54mm_Vertical, F.Cu at (338.6, 29.6)
- added L201: 1u, Inductor_SMD:L_1812_4532Metric, F.Cu at (350.3, 136.0)
- added L202: 1u, Inductor_SMD:L_1812_4532Metric, F.Cu at (340.1, 148.4)
- added L203: 1u, Inductor_SMD:L_1812_4532Metric, F.Cu at (343.3, 140.9)
- added L204: 1u, Inductor_SMD:L_1812_4532Metric, F.Cu at (343.3, 136.0)
- added L301: 1u, Inductor_SMD:L_1812_4532Metric, F.Cu at (408.2, 52.2)
- added L302: 1u, Inductor_SMD:L_1812_4532Metric, F.Cu at (401.2, 52.2)
- added L303: 1u, Inductor_SMD:L_1812_4532Metric, F.Cu at (398.0, 64.7)
- added L304: 1u, Inductor_SMD:L_1812_4532Metric, F.Cu at (401.2, 57.2)
- added L401: 1u, Inductor_SMD:L_1812_4532Metric, F.Cu at (363.5, 86.4)
- added L402: 1u, Inductor_SMD:L_1812_4532Metric, F.Cu at (360.3, 93.9)
- added L403: 1u, Inductor_SMD:L_1812_4532Metric, F.Cu at (370.5, 81.5)
- added L404: 1u, Inductor_SMD:L_1812_4532Metric, F.Cu at (363.5, 81.5)
- added L501: 1u, Inductor_SMD:L_1812_4532Metric, F.Cu at (420.1, 29.7)
- added L502: 1u, Inductor_SMD:L_1812_4532Metric, F.Cu at (410.0, 42.2)
- added L503: 1u, Inductor_SMD:L_1812_4532Metric, F.Cu at (413.2, 29.7)
- added L504: 1u, Inductor_SMD:L_1812_4532Metric, F.Cu at (413.2, 34.7)
- added L601: 1u, Inductor_SMD:L_1812_4532Metric, F.Cu at (370.5, 59.0)
- added L602: 1u, Inductor_SMD:L_1812_4532Metric, F.Cu at (360.3, 71.4)
- added L603: 1u, Inductor_SMD:L_1812_4532Metric, F.Cu at (363.5, 63.9)
- added L604: 1u, Inductor_SMD:L_1812_4532Metric, F.Cu at (363.5, 59.0)
- added L701: 1u, Inductor_SMD:L_1812_4532Metric, F.Cu at (332.8, 81.5)
- added L702: 1u, Inductor_SMD:L_1812_4532Metric, F.Cu at (325.9, 81.5)
- added L703: 1u, Inductor_SMD:L_1812_4532Metric, F.Cu at (325.9, 86.4)
- added L704: 1u, Inductor_SMD:L_1812_4532Metric, F.Cu at (322.7, 93.9)
- added L801: 1u, Inductor_SMD:L_1812_4532Metric, F.Cu at (382.5, 29.7)
- added L802: 1u, Inductor_SMD:L_1812_4532Metric, F.Cu at (372.3, 42.2)
- added L803: 1u, Inductor_SMD:L_1812_4532Metric, F.Cu at (375.5, 34.7)
- added L804: 1u, Inductor_SMD:L_1812_4532Metric, F.Cu at (375.5, 29.7)
- added L901: 1u, Inductor_SMD:L_1812_4532Metric, F.Cu at (322.7, 71.4)
- added L902: 1u, Inductor_SMD:L_1812_4532Metric, F.Cu at (325.9, 59.0)
- added L903: 1u, Inductor_SMD:L_1812_4532Metric, F.Cu at (332.8, 59.0)
- added L904: 1u, Inductor_SMD:L_1812_4532Metric, F.Cu at (325.9, 63.9)
- added Q101: NTR5103NT1G, Package_TO_SOT_SMD:SOT-23, F.Cu at (333.9, 41.3)
- added Q102: RSC002P03T316, Package_TO_SOT_SMD:SOT-23, F.Cu at (338.3, 36.7)
- added Q103: RSC002P03T316, Package_TO_SOT_SMD:SOT-23, F.Cu at (333.9, 36.7)
- added Q104: NTR5103NT1G, Package_TO_SOT_SMD:SOT-23, F.Cu at (343.2, 29.5)
- added Q201: NTR5103NT1G, Package_TO_SOT_SMD:SOT-23, F.Cu at (356.0, 135.8)
- added Q202: NTR5103NT1G, Package_TO_SOT_SMD:SOT-23, F.Cu at (349.0, 140.7)
- added Q301: NTR5103NT1G, Package_TO_SOT_SMD:SOT-23, F.Cu at (406.9, 57.0)
- added Q302: NTR5103NT1G, Package_TO_SOT_SMD:SOT-23, F.Cu at (413.9, 52.0)
- added Q401: NTR5103NT1G, Package_TO_SOT_SMD:SOT-23, F.Cu at (369.2, 86.2)
- added Q402: NTR5103NT1G, Package_TO_SOT_SMD:SOT-23, F.Cu at (376.2, 81.3)
- added Q501: NTR5103NT1G, Package_TO_SOT_SMD:SOT-23, F.Cu at (425.8, 29.5)
- added Q502: NTR5103NT1G, Package_TO_SOT_SMD:SOT-23, F.Cu at (418.9, 34.5)
- added Q601: NTR5103NT1G, Package_TO_SOT_SMD:SOT-23, F.Cu at (369.2, 63.7)
- added Q602: NTR5103NT1G, Package_TO_SOT_SMD:SOT-23, F.Cu at (376.2, 58.8)
- added Q701: NTR5103NT1G, Package_TO_SOT_SMD:SOT-23, F.Cu at (331.6, 86.2)
- added Q702: NTR5103NT1G, Package_TO_SOT_SMD:SOT-23, F.Cu at (338.5, 81.3)
- added Q801: NTR5103NT1G, Package_TO_SOT_SMD:SOT-23, F.Cu at (381.2, 34.5)
- added Q802: NTR5103NT1G, Package_TO_SOT_SMD:SOT-23, F.Cu at (388.2, 29.5)
- added Q901: NTR5103NT1G, Package_TO_SOT_SMD:SOT-23, F.Cu at (338.5, 58.8)
- added Q902: NTR5103NT1G, Package_TO_SOT_SMD:SOT-23, F.Cu at (331.6, 63.7)
- added R101: 10k, Resistor_SMD:R_0805_2012Metric, F.Cu at (334.5, 50.9)
- added R102: 10k, Resistor_SMD:R_0805_2012Metric, F.Cu at (352.0, 34.6)
- added R103: 100k, Resistor_SMD:R_0805_2012Metric, F.Cu at (347.1, 40.5)
- added R201: 150R, Resistor_SMD:R_0805_2012Metric, F.Cu at (350.2, 150.4)
- added R202: 150R, Resistor_SMD:R_0805_2012Metric, F.Cu at (354.6, 145.9)
- added R203: 100k, Resistor_SMD:R_0805_2012Metric, F.Cu at (354.6, 143.0)
- added R204: 10k, Resistor_SMD:R_0805_2012Metric, F.Cu at (357.9, 139.5)
- added R205: 100k, Resistor_SMD:R_0805_2012Metric, F.Cu at (350.2, 144.5)
- added R206: 10k, Resistor_SMD:R_0805_2012Metric, F.Cu at (345.8, 147.9)
- added R301: 150R, Resistor_SMD:R_0805_2012Metric, F.Cu at (417.0, 61.7)
- added R302: 150R, Resistor_SMD:R_0805_2012Metric, F.Cu at (415.8, 55.8)
- added R303: 100k, Resistor_SMD:R_0805_2012Metric, F.Cu at (403.7, 67.1)
- added R304: 10k, Resistor_SMD:R_0805_2012Metric, F.Cu at (412.6, 62.2)
- added R305: 100k, Resistor_SMD:R_0805_2012Metric, F.Cu at (412.6, 59.2)
- added R306: 10k, Resistor_SMD:R_0805_2012Metric, F.Cu at (408.1, 63.7)
- added R401: 150R, Resistor_SMD:R_0805_2012Metric, F.Cu at (379.3, 90.9)
- added R402: 150R, Resistor_SMD:R_0805_2012Metric, F.Cu at (366.0, 93.4)
- added R403: 100k, Resistor_SMD:R_0805_2012Metric, F.Cu at (378.1, 85.0)
- added R404: 10k, Resistor_SMD:R_0805_2012Metric, F.Cu at (366.0, 96.4)
- added R405: 100k, Resistor_SMD:R_0805_2012Metric, F.Cu at (370.5, 92.9)
- added R406: 10k, Resistor_SMD:R_0805_2012Metric, F.Cu at (379.3, 88.0)
- added R501: 150R, Resistor_SMD:R_0805_2012Metric, F.Cu at (427.8, 33.3)
- added R502: 150R, Resistor_SMD:R_0805_2012Metric, F.Cu at (420.1, 38.2)
- added R503: 100k, Resistor_SMD:R_0805_2012Metric, F.Cu at (415.7, 41.7)
- added R504: 10k, Resistor_SMD:R_0805_2012Metric, F.Cu at (424.5, 36.7)
- added R505: 100k, Resistor_SMD:R_0805_2012Metric, F.Cu at (415.7, 44.6)
- added R506: 10k, Resistor_SMD:R_0805_2012Metric, F.Cu at (420.1, 41.2)
- added R601: 150R, Resistor_SMD:R_0805_2012Metric, F.Cu at (374.9, 71.9)
- added R602: 150R, Resistor_SMD:R_0805_2012Metric, F.Cu at (379.3, 65.5)
- added R603: 100k, Resistor_SMD:R_0805_2012Metric, F.Cu at (370.4, 73.4)
- added R604: 10k, Resistor_SMD:R_0805_2012Metric, F.Cu at (370.5, 67.5)
- added R605: 100k, Resistor_SMD:R_0805_2012Metric, F.Cu at (374.9, 68.9)
- added R606: 10k, Resistor_SMD:R_0805_2012Metric, F.Cu at (374.9, 66.0)
- added R701: 150R, Resistor_SMD:R_0805_2012Metric, F.Cu at (332.8, 90.0)
- added R702: 150R, Resistor_SMD:R_0805_2012Metric, F.Cu at (341.6, 88.0)
- added R703: 100k, Resistor_SMD:R_0805_2012Metric, F.Cu at (328.3, 93.4)
- added R704: 10k, Resistor_SMD:R_0805_2012Metric, F.Cu at (340.4, 85.0)
- added R705: 100k, Resistor_SMD:R_0805_2012Metric, F.Cu at (328.3, 96.4)
- added R706: 10k, Resistor_SMD:R_0805_2012Metric, F.Cu at (332.8, 92.9)
- added R801: 150R, Resistor_SMD:R_0805_2012Metric, F.Cu at (386.8, 39.7)
- added R802: 150R, Resistor_SMD:R_0805_2012Metric, F.Cu at (378.0, 41.7)
- added R803: 100k, Resistor_SMD:R_0805_2012Metric, F.Cu at (390.1, 33.3)
- added R804: 10k, Resistor_SMD:R_0805_2012Metric, F.Cu at (378.0, 44.6)
- added R805: 100k, Resistor_SMD:R_0805_2012Metric, F.Cu at (391.2, 39.2)
- added R806: 10k, Resistor_SMD:R_0805_2012Metric, F.Cu at (386.8, 42.6)
- added R901: 150R, Resistor_SMD:R_0805_2012Metric, F.Cu at (340.4, 62.5)
- added R902: 150R, Resistor_SMD:R_0805_2012Metric, F.Cu at (328.3, 73.9)
- added R903: 100k, Resistor_SMD:R_0805_2012Metric, F.Cu at (332.8, 70.4)
- added R904: 10k, Resistor_SMD:R_0805_2012Metric, F.Cu at (337.2, 66.0)
- added R905: 100k, Resistor_SMD:R_0805_2012Metric, F.Cu at (337.2, 68.9)
- added R906: 10k, Resistor_SMD:R_0805_2012Metric, F.Cu at (332.7, 73.4)
- added U201: Opamp_Quad_Generic, Package_SO:TSSOP-14_4.4x5mm_P0.65mm, F.Cu at (332.2, 149.2)
- added U301: Opamp_Quad_Generic, Package_SO:TSSOP-14_4.4x5mm_P0.65mm, F.Cu at (390.1, 65.5)
- added U401: Opamp_Quad_Generic, Package_SO:TSSOP-14_4.4x5mm_P0.65mm, F.Cu at (352.4, 94.8)
- added U501: Opamp_Quad_Generic, Package_SO:TSSOP-14_4.4x5mm_P0.65mm, F.Cu at (402.0, 43.0)
- added U601: Opamp_Quad_Generic, Package_SO:TSSOP-14_4.4x5mm_P0.65mm, F.Cu at (352.4, 72.3)
- added U701: Opamp_Quad_Generic, Package_SO:TSSOP-14_4.4x5mm_P0.65mm, F.Cu at (314.7, 94.8)
- added U801: Opamp_Quad_Generic, Package_SO:TSSOP-14_4.4x5mm_P0.65mm, F.Cu at (364.3, 43.0)
- added U901: Opamp_Quad_Generic, Package_SO:TSSOP-14_4.4x5mm_P0.65mm, F.Cu at (314.7, 72.3)
