File: Malfunctionboard.kicad_pcb (KiCad board)
At the start: 2 copper layers, 141.4 x 32.7 mm, 266 parts, among them J1 In/out, J2 In/out, J201 Conn_Coaxial, J202 Conn_Coaxial, J301 Conn_Coaxial, J302 Conn_Coaxial, J401 Conn_Coaxial, J402 Conn_Coaxial, J501 Conn_Coaxial, J502 Conn_Coaxial, J601 Conn_Coaxial, J602 Conn_Coaxial, J701 Conn_Coaxial, J702 Conn_Coaxial, J801 Conn_Coaxial, J802 Conn_Coaxial, J901 Conn_Coaxial, J902 Conn_Coaxial, Q1 RSC002P03T316, Q2 RSC002P03T316, Q201 NTR5103NT1G, Q202 NTR5103NT1G, Q3 RSC002P03T316, Q301 NTR5103NT1G, Q302 NTR5103NT1G, Q401 NTR5103NT1G, Q402 NTR5103NT1G, Q501 NTR5103NT1G, Q502 NTR5103NT1G, Q601 NTR5103NT1G, Q602 NTR5103NT1G, Q701 NTR5103NT1G, Q702 NTR5103NT1G, Q801 NTR5103NT1G, Q802 NTR5103NT1G, Q901 NTR5103NT1G, Q902 NTR5103NT1G, U201 LM339PW, U301 LM339PW, U401 LM339PW, U501 LM339PW, U601 LM339PW, U701 LM339PW, U801 LM339PW, U901 LM339PW

Commit message: Updated to v1.0
Other:
- rule pad_to_mask_clearance: 0.051 -> 0
- board text added: "04/2020 v1.0"
- board text added: "Malfunctionboard v1.0"
- board text removed: "04/2020 v0.3"
- board text removed: "Malfunctionboard v0.3"

Commit message: Updated version date
Other:
- board text added: "11/2021 v1.0"
- board text removed: "04/2020 v1.0"
